Commit message: modified:   config/md_rviz.rviz 	modified:   description/md.urdf.xacro     modified:   description/md_core.xacro

File: description/md.urdf.xacro (robot description, xacro)
@@ -4,4 +4,4 @@
     <xacro:include filename="lidar.xacro"/>
     <xacro:include filename="md_core.xacro"/>
-    <xacro:include filename="gazebo_control.xacro"/>
+    <!-- <xacro:include filename="gazebo_control.xacro"/> -->
 </robot>

File: description/md_core.xacro (robot description, xacro)
@@ -172,9 +172,35 @@
         <material>Gazebo/Blue</material>
     </gazebo>
+    <!-- REAR AXEL LINK -->
+    <joint name="rear_axel_joint" type="continuous">
+        <parent link="base_link"/>
+        <child link="rear_axel"/>
+        <origin xyz="-0.945 0 0" rpy="-${pi/2} 0 0" />
+        <axis xyz="0 0 1"/>
+    </joint>
+    <link name="rear_axel">
+        <visual>
+            <geometry>
+                <cylinder radius="0.005" length="0.2202"/>
+            </geometry>
+            <material name="blue"/>
+        </visual>
+        <collision>
+            <geometry>
+                <sphere radius="${rear_wheel_radius}"/>
+            </geometry>
+        </collision>
+        <xacro:inertial_cylinder mass="${wheel_mass}" length="${rear_wheel_thickness}" radius="${rear_wheel_radius}">
+            <origin xyz="0 0 0" rpy="0 0 0"/>
+        </xacro:inertial_cylinder>
+    </link>
+    <gazebo reference="rear_left_wheel">
+        <material>Gazebo/Red</material>
+    </gazebo>
     <!-- REAR LEFT WHEEL LINK -->
-    <joint name="rear_left_wheel_joint" type="continuous">
-        <parent link="base_link"/>
+    <joint name="rear_left_wheel_joint" type="fixed">
+        <parent link="rear_axel"/>
         <child link="rear_left_wheel"/>
-        <origin xyz="-0.945 ${rear_wheel_offset_y} 0" rpy="-${pi/2} 0 0" />
+        <origin xyz="0 0 ${rear_wheel_offset_y}" rpy="0 0 0" />
         <axis xyz="0 0 1"/>
     </joint>
@@ -199,8 +225,8 @@
     </gazebo>
 <!-- REAR RIGHT WHEEL LINK -->
-    <joint name="rear_right_wheel_joint" type="continuous">
-        <parent link="base_link"/>
+    <joint name="rear_right_wheel_joint" type="fixed">
+        <parent link="rear_axel"/>
         <child link="rear_right_wheel"/>
-        <origin xyz="-0.945 ${-rear_wheel_offset_y} 0" rpy="${pi/2} 0 0" />
+        <origin xyz="0 0 ${-rear_wheel_offset_y}" rpy="0 0 0" />
         <axis xyz="0 0 -1"/>
     </joint>
