Commit message: modified:   description/md_core.xacro

File: description/md_core.xacro (robot description, xacro)
@@ -188,12 +188,12 @@
         <collision>
             <geometry>
-                <sphere radius="${rear_wheel_radius}"/>
-            </geometry>
-        </collision>
-        <xacro:inertial_cylinder mass="${wheel_mass}" length="${rear_wheel_thickness}" radius="${rear_wheel_radius}">
-            <origin xyz="0 0 0" rpy="0 0 0"/>
-        </xacro:inertial_cylinder>
-    </link>
-    <gazebo reference="rear_left_wheel">
+                <cylinder radius="${rear_wheel_radius}"/>
+            </geometry>
+        </collision>
+        <xacro:inertial_cylinder mass="${wheel_mass}" length="0.2202" radius="0.005">
+            <origin xyz="0 0 0" rpy="0 0 0"/>
+        </xacro:inertial_cylinder>
+    </link>
+    <gazebo reference="rear_axel">
         <material>Gazebo/Red</material>
     </gazebo>

Commit message: modified:   description/md_core.xacro 	modified:   launch/steering.launch.py 	modified:   scripts/wheel_steer.py

File: description/md_core.xacro (robot description, xacro)
@@ -11,7 +11,7 @@
     <xacro:property name="rear_wheel_thickness" value="0.061"/>
     <xacro:property name="wheel_mass" value="0.05"/>
-    <xacro:property name="front_wheel_offset_y" value="0.0819"/>
-    <xacro:property name="rear_wheel_offset_y" value="0.1101"/>
-    <xacro:property name="rear_wheel_offset_x" value="-0.945"/>
+    <xacro:property name="front_wheel_offset_y" value="0.082"/>
+    <xacro:property name="rear_wheel_offset_y" value="0.11"/>
+    <xacro:property name="rear_wheel_offset_x" value="-0.8817"/>
     <xacro:property name="steer_limlow" value="-.785398"/>
     <xacro:property name="steer_limhigh" value="0.785398"/>
@@ -74,5 +74,5 @@
         <parent link="base_link"/>
         <child link="front_left_axel"/>
-        <origin xyz="-0.5375 ${front_wheel_offset_y - 0.0319} 0" rpy="-${pi/2} 0 0" />
+        <origin xyz="-0.5543 ${front_wheel_offset_y - 0.0319} 0" rpy="-${pi/2} 0 0" />
         <axis xyz="0 -1 0"/>
         <limit lower="${-pi/4}" upper="${pi/4}" velocity="100" effort="100"/>
@@ -129,5 +129,5 @@
         <parent link="base_link"/>
         <child link="front_right_axel"/>
-        <origin xyz="-0.5375 ${-front_wheel_offset_y + 0.0319} 0" rpy="-${pi/2} 0 0" />
+        <origin xyz="-0.5543 ${-front_wheel_offset_y + 0.0319} 0" rpy="-${pi/2} 0 0" />
         <axis xyz="0 1 0"/>
         <limit lower="${-pi/4}" upper="${pi/4}" velocity="100" effort="100"/>
