Commit message: new file:   config/controller_configuration.yaml 	modified:   description/gazebo_control.xacro 	modified:   description/md.urdf.xacro 	modified:   description/md_core.xacro

File: description/gazebo_control.xacro (robot description, xacro)
@@ -1,42 +1,28 @@
 <?xml version="1.0"?>
 <robot xmlns:xacro="https://www.ros.org/wiki/xacro">
+    <ros2_control name="GazeboSystem" type="system">
+        <hardware>
+            <plugin>gazebo_ros2_control/GazeboSystem/<plugin>
+        </hardware>
+        <joint_name="front_right_axel_joint">
+            <command_interface name="position">
+                <param name="min">${steer_limlow}</param>
+                <param name="max">${steer_limhigh}</param>
+            </command_interface>
+            <state_interface name="position"/>
+            <state_interface name="velocity"/>
+        </joint>
+        <joint_name="front_left_axel_joint">
+            <command_interface name="position">
+                <param name="min">${steer_limlow}</param>
+                <param name="max">${steer_limhigh}</param>
+            </command_interface>
+            <state_interface name="position"/>
+            <state_interface name="velocity"/>
+        </joint>
+    </ros2_control>
     <gazebo>
-        <plugin name="gazebo_ros_ackermann_drive" filename="libgazebo_ros_ackermann_drive.so">
-        <ros>
-            <namespace>demo</namespace>
-            <remapping>cmd_vel:=cmd_demo</remapping>
-            <remapping>odom:=odom_demo</remapping>
-            <remapping>distance:=distance_demo</remapping>
-        </ros>
-        <update_rate>100.0</update_rate>
-        <!-- wheels -->
-        <front_left_joint>front_left_wheel_joint</front_left_joint>
-        <front_right_joint>front_right_wheel_joint</front_right_joint>
-        <rear_left_joint>rear_left_wheel_joint</rear_left_joint>
-        <rear_right_joint>rear_right_wheel_joint</rear_right_joint>
-        <left_steering_joint>front_left_axel_joint</left_steering_joint>
-        <right_steering_joint>front_right_axel_joint</right_steering_joint>
-        <!--<steering_wheel_joint>steering_joint</steering_wheel_joint> -->
-        <!-- Max absolute steer angle for tyre in radians-->
-        <!-- Any cmd_vel angular z greater than this would be capped -->
-        <max_steer>0.6458</max_steer>
-        <!-- Max absolute steering angle of steering wheel -->
-        <!--<max_steering_angle>7.85</max_steering_angle> -->
-        <!-- Max absolute linear speed in m/s -->
-        <max_speed>20</max_speed>
-        <!-- PID tuning -->
-        <left_steering_pid_gain>1500 0 1</left_steering_pid_gain>
-        <left_steering_i_range>0 0</left_steering_i_range>
-        <right_steering_pid_gain>1500 0 1</right_steering_pid_gain>
-        <right_steering_i_range>0 0</right_steering_i_range>
-        <linear_velocity_pid_gain>1000 0 1</linear_velocity_pid_gain>
-        <linear_velocity_i_range>0 0</linear_velocity_i_range>
-        <!-- output -->
-        <publish_odom>true</publish_odom>
-        <publish_odom_tf>true</publish_odom_tf>
-        <publish_wheel_tf>true</publish_wheel_tf>
-        <publish_distance>true</publish_distance>
-        <odometry_frame>odom_demo</odometry_frame>
-        <robot_base_frame>base_link</robot_base_frame>
+        <plugin filename="libgazebo_ros2_control.so" name"gazebo_ros2_control">
+            <parameters>$(find md_beta)/config/controller_configuration.yaml</parameters>
         </plugin>
     </gazebo>

File: description/md.urdf.xacro (robot description, xacro)
@@ -4,4 +4,4 @@
     <xacro:include filename="lidar.xacro"/>
     <xacro:include filename="md_core.xacro"/>
-    <!-- <xacro:include filename="gazebo_control.xacro"/> -->
+    <xacro:include filename="gazebo_control.xacro"/>
 </robot>

File: description/md_core.xacro (robot description, xacro)
@@ -188,5 +188,5 @@
         <collision>
             <geometry>
-                <cylinder radius="${rear_wheel_radius}"/>
+                <cylinder radius="${rear_wheel_radius}" length="0.2202"/>
             </geometry>
         </collision>

Commit message: modified:   CMakeLists.txt 	modified:   description/gazebo_control.xacro 	modified:   launch/launch_sim.launch.py 	new file:   launch/my_robot.launch.py 	new file:   launch/steering.launch.py

File: description/gazebo_control.xacro (robot description, xacro)
@@ -1,9 +1,13 @@
 <?xml version="1.0"?>
 <robot xmlns:xacro="https://www.ros.org/wiki/xacro">
+   <!-- Properties -->
+	   <xacro:property name="PI" value="3.1415926535897931"/>
+	   <xacro:property name="steer_limlow" value="-0.7854"/>
+	   <xacro:property name="steer_limhigh" value="0.7854"/>
     <ros2_control name="GazeboSystem" type="system">
         <hardware>
-            <plugin>gazebo_ros2_control/GazeboSystem/<plugin>
+            <plugin>gazebo_ros2_control/GazeboSystem</plugin>
         </hardware>
-        <joint_name="front_right_axel_joint">
+        <joint name="front_right_axel_joint">
             <command_interface name="position">
                 <param name="min">${steer_limlow}</param>
@@ -13,5 +17,5 @@
             <state_interface name="velocity"/>
         </joint>
-        <joint_name="front_left_axel_joint">
+        <joint name="front_left_axel_joint">
             <command_interface name="position">
                 <param name="min">${steer_limlow}</param>
@@ -23,5 +27,5 @@
     </ros2_control>
     <gazebo>
-        <plugin filename="libgazebo_ros2_control.so" name"gazebo_ros2_control">
+        <plugin filename="libgazebo_ros2_control.so" name="gazebo_ros2_control">
             <parameters>$(find md_beta)/config/controller_configuration.yaml</parameters>
         </plugin>

Commit message: modified:   config/controller_configuration.yaml     modified:   description/gazebo_control.xacro 	modified:   description/md_core.xacro 	modified:   scripts/wheel_steer.py

File: description/gazebo_control.xacro (robot description, xacro)
@@ -3,6 +3,6 @@
    <!-- Properties -->
 	   <xacro:property name="PI" value="3.1415926535897931"/>
-	   <xacro:property name="steer_limlow" value="-0.7854"/>
-	   <xacro:property name="steer_limhigh" value="0.7854"/>
+	   <xacro:property name="steer_limlow" value="${-pi/4}"/>
+	   <xacro:property name="steer_limhigh" value="${pi/4}"/>
     <ros2_control name="GazeboSystem" type="system">
         <hardware>

File: description/md_core.xacro (robot description, xacro)
@@ -65,4 +65,5 @@
     <gazebo reference="chassis">
         <material>Gazebo/Orange</material>
+        <dynamics damping="0.7"/>
     </gazebo>
     <!-- FRONT LEFT AXEL LINK-->
@@ -118,4 +119,6 @@
     <gazebo reference="front_left_wheel">
         <material>Gazebo/Blue</material>
+        <mu1 value="0.001"/>
+        <mu2 value="0.001"/>
     </gazebo>
   <!-- FRONT RIGHT AXEL LINK-->
@@ -171,4 +174,6 @@
     <gazebo reference="front_right_wheel">
         <material>Gazebo/Blue</material>
+        <mu1 value="0.001"/>
+        <mu2 value="0.001"/>
     </gazebo>
     <!-- REAR AXEL LINK -->

Commit message: new file:   scripts/__init__.py

File: description/gazebo_control.xacro (robot description, xacro)
@@ -25,8 +25,24 @@
             <state_interface name="velocity"/>
         </joint>
+        <joint name="rear_left_wheel_joint">
+            <command_interface name="velocity">
+                <param name="min">-10</param>
+                <param name="max">10</param>
+            </command_interface>
+            <state_interface name="velocity"/>
+            <state_interface name="position"/>
+        </joint>
+        <joint name="rear_right_wheel_joint">
+            <command_interface name="velocity">
+                <param name="min">-10</param>
+                <param name="max">10</param>
+            </command_interface>
+            <state_interface name="velocity"/>
+            <state_interface name="position"/>
+        </joint>
     </ros2_control>
     <gazebo>
         <plugin filename="libgazebo_ros2_control.so" name="gazebo_ros2_control">
-            <parameters>$(find md_beta)/config/controller_configuration.yaml</parameters>
+            <parameters>$(find rmd_beta)/config/controller_configuration.yaml</parameters>
         </plugin>
     </gazebo>

File: description/lidar.xacro (robot description, xacro)
@@ -50,5 +50,5 @@
             <plugin name="laser_controller" filename="libgazebo_ros_ray_sensor.so">
                 <ros>
-                    <argument>--ros-args --remap ~/out:=scan</argument>
+                    <argument>~/out:=scan</argument>
                 </ros>
                 <output_type>sensor_msgs/LaserScan</output_type>

File: description/md_core.xacro (robot description, xacro)
@@ -13,4 +13,7 @@
     <xacro:property name="front_wheel_offset_y" value="0.0819"/>
     <xacro:property name="rear_wheel_offset_y" value="0.1101"/>
+    <xacro:property name="rear_wheel_offset_x" value="-0.945"/>
+    <xacro:property name="steer_limlow" value="-.785398"/>
+    <xacro:property name="steer_limhigh" value="0.785398"/>
     <material name="white">
         <color rgba="1 1 1 1" />
@@ -95,5 +98,5 @@
     </gazebo>
     <!-- FRONT LEFT WHEEL LINK -->
-    <joint name="front_left_wheel_joint" type="continuous">
+    <joint name="front_left_wheel_joint" type="fixed">
         <parent link="front_left_axel"/>
         <child link="front_left_wheel"/>
@@ -119,6 +122,6 @@
     <gazebo reference="front_left_wheel">
         <material>Gazebo/Blue</material>
-        <mu1 value="0.001"/>
-        <mu2 value="0.001"/>
+        <!-- <mu1 value="0.001"/>
+        <mu2 value="0.001"/> -->
     </gazebo>
   <!-- FRONT RIGHT AXEL LINK-->
@@ -150,5 +153,5 @@
     </gazebo>
     <!-- FRONT RIGHT WHEEL LINK -->
-    <joint name="front_right_wheel_joint" type="continuous">
+    <joint name="front_right_wheel_joint" type="fixed">
         <parent link="front_right_axel"/>
         <child link="front_right_wheel"/>
@@ -174,40 +177,14 @@
     <gazebo reference="front_right_wheel">
         <material>Gazebo/Blue</material>
-        <mu1 value="0.001"/>
-        <mu2 value="0.001"/>
-    </gazebo>
-    <!-- REAR AXEL LINK -->
-    <joint name="rear_axel_joint" type="continuous">
-        <parent link="base_link"/>
-        <child link="rear_axel"/>
-        <origin xyz="-0.945 0 0" rpy="-${pi/2} 0 0" />
+        <!-- <mu1 value="0.001"/>
+        <mu2 value="0.001"/> -->
+    </gazebo>
+    <!-- REAR LEFT WHEEL LINK -->
+    <joint name="rear_left_wheel_joint" type="continuous">
+        <parent link="base_link"/>
+        <child link="rear_left_wheel"/>
+        <origin xyz="${rear_wheel_offset_x} ${rear_wheel_offset_y} 0" rpy="-${pi/2} 0 0" />
         <axis xyz="0 0 1"/>
     </joint>
-    <link name="rear_axel">
-        <visual>
-            <geometry>
-                <cylinder radius="0.005" length="0.2202"/>
-            </geometry>
-            <material name="blue"/>
-        </visual>
-        <collision>
-            <geometry>
-                <cylinder radius="${rear_wheel_radius}" length="0.2202"/>
-            </geometry>
-        </collision>
-        <xacro:inertial_cylinder mass="${wheel_mass}" length="0.2202" radius="0.005">
-            <origin xyz="0 0 0" rpy="0 0 0"/>
-        </xacro:inertial_cylinder>
-    </link>
-    <gazebo reference="rear_axel">
-        <material>Gazebo/Red</material>
-    </gazebo>
-    <!-- REAR LEFT WHEEL LINK -->
-    <joint name="rear_left_wheel_joint" type="fixed">
-        <parent link="rear_axel"/>
-        <child link="rear_left_wheel"/>
-        <origin xyz="0 0 ${rear_wheel_offset_y}" rpy="0 0 0" />
-        <axis xyz="0 0 1"/>
-    </joint>
     <link name="rear_left_wheel">
         <visual>
@@ -230,8 +207,8 @@
     </gazebo>
 <!-- REAR RIGHT WHEEL LINK -->
-    <joint name="rear_right_wheel_joint" type="fixed">
-        <parent link="rear_axel"/>
+    <joint name="rear_right_wheel_joint" type="continuous">
+        <parent link="base_link"/>
         <child link="rear_right_wheel"/>
-        <origin xyz="0 0 ${-rear_wheel_offset_y}" rpy="0 0 0" />
+        <origin xyz="${rear_wheel_offset_x} ${-rear_wheel_offset_y} 0" rpy="${pi/2} 0 0" />
         <axis xyz="0 0 -1"/>
     </joint>

Commit message: modified:   config/controller_configuration.yaml 	new file:   config/mapper_params_online_async.yaml 	modified:   config/md_rviz.rviz 	modified:   description/gazebo_control.xacro 	modified:   description/lidar.xacro 	modified:   description/md_core.xacro 	modified:   launch/launch_sim.launch.py 	modified:   launch/rsp.launch.py 	modified:   package.xml 	modified:   scripts/wheel_steer.py 	modified:   worlds/obstacles.world

File: description/gazebo_control.xacro (robot description, xacro)
@@ -1,8 +1,4 @@
 <?xml version="1.0"?>
 <robot xmlns:xacro="https://www.ros.org/wiki/xacro">
-   <!-- Properties -->
-	   <xacro:property name="PI" value="3.1415926535897931"/>
-	   <xacro:property name="steer_limlow" value="${-pi/4}"/>
-	   <xacro:property name="steer_limhigh" value="${pi/4}"/>
     <ros2_control name="GazeboSystem" type="system">
         <hardware>
@@ -45,4 +41,9 @@
         <plugin filename="libgazebo_ros2_control.so" name="gazebo_ros2_control">
             <parameters>$(find rmd_beta)/config/controller_configuration.yaml</parameters>
+            <odometry_frame>odom</odometry_frame>
+            <robot_base_frame>base_link</robot_base_frame>
+            <publish_odom>true</publish_odom>
+            <publish_odom_tf>true</publish_odom_tf>
+            <publish_wheel_tf>true</publish_wheel_tf>
         </plugin>
     </gazebo>

File: description/md_core.xacro (robot description, xacro)
@@ -91,5 +91,5 @@
         </collision>
         <xacro:inertial_cylinder mass="0.005" length="0.0319" radius="0.005">
-            <origin xyz="0 0 0" rpy="0 0 0"/>
+            <origin xyz="0 0 1" rpy="0 0 0"/>
         </xacro:inertial_cylinder>
     </link>
@@ -129,5 +129,5 @@
         <parent link="base_link"/>
         <child link="front_right_axel"/>
-        <origin xyz="-0.5543 ${-front_wheel_offset_y + 0.0319} 0" rpy="-${pi/2} 0 0" />
+        <origin xyz="-0.5543 ${-front_wheel_offset_y + 0.0319} 0" rpy="${pi/2} 0 0" />
         <axis xyz="0 1 0"/>
         <limit lower="${-pi/4}" upper="${pi/4}" velocity="100" effort="100"/>
@@ -156,5 +156,5 @@
         <parent link="front_right_axel"/>
         <child link="front_right_wheel"/>
-        <origin xyz="0 0 -0.0319" rpy="0 0 0" />
+        <origin xyz="0 0 0.0319" rpy="0 0 0" />
         <axis xyz="0 0 -1"/>
     </joint>

Commit message: modified:   description/gazebo_control.xacro 	modified:   description/md_core.xacro 	modified:   launch/launch_sim.launch.py 	modified:   package.xml

File: description/gazebo_control.xacro (robot description, xacro)
@@ -41,9 +41,4 @@
         <plugin filename="libgazebo_ros2_control.so" name="gazebo_ros2_control">
             <parameters>$(find rmd_beta)/config/controller_configuration.yaml</parameters>
-            <odometry_frame>odom</odometry_frame>
-            <robot_base_frame>base_link</robot_base_frame>
-            <publish_odom>true</publish_odom>
-            <publish_odom_tf>true</publish_odom_tf>
-            <publish_wheel_tf>true</publish_wheel_tf>
         </plugin>
     </gazebo>

File: description/md_core.xacro (robot description, xacro)
@@ -70,39 +70,13 @@
         <dynamics damping="0.7"/>
     </gazebo>
-    <!-- FRONT LEFT AXEL LINK-->
-    <joint name="front_left_axel_joint" type="revolute">
+    <!-- FRONT WHEEL LINK -->
+    <joint name="front_wheel_joint" type="revolute">
         <parent link="base_link"/>
-        <child link="front_left_axel"/>
-        <origin xyz="-0.5543 ${front_wheel_offset_y - 0.0319} 0" rpy="-${pi/2} 0 0" />
-        <axis xyz="0 -1 0"/>
+        <child link="front_wheel"/>
+        <origin xyz="-0.5543 0 0" rpy="${pi/2} 0 0" />
+        <axis xyz="0 1 0"/>
         <limit lower="${-pi/4}" upper="${pi/4}" velocity="100" effort="100"/>
     </joint>
-    <link name="front_left_axel">
-        <visual>
-            <geometry>
-                <cylinder radius="0.005" length="0.0319"/>
-            </geometry>
-            <material name="red"/>
-        </visual>
-        <collision>
-            <geometry>
-                <sphere radius="0.005"/>
-            </geometry>
-        </collision>
-        <xacro:inertial_cylinder mass="0.005" length="0.0319" radius="0.005">
-            <origin xyz="0 0 1" rpy="0 0 0"/>
-        </xacro:inertial_cylinder>
-    </link>
-    <gazebo reference="front_left_axel">
-        <material>Gazebo/Red</material>
-    </gazebo>
-    <!-- FRONT LEFT WHEEL LINK -->
-    <joint name="front_left_wheel_joint" type="fixed">
-        <parent link="front_left_axel"/>
-        <child link="front_left_wheel"/>
-        <origin xyz="0 0 0.0319" rpy="0 0 0" />
-        <axis xyz="0 0 1"/>
-    </joint>
-    <link name="front_left_wheel">
+    <link name="front_wheel">
         <visual>
             <geometry>
@@ -120,60 +94,5 @@
         </xacro:inertial_cylinder>
     </link>
-    <gazebo reference="front_left_wheel">
-        <material>Gazebo/Blue</material>
-        <!-- <mu1 value="0.001"/>
-        <mu2 value="0.001"/> -->
-    </gazebo>
-  <!-- FRONT RIGHT AXEL LINK-->
-    <joint name="front_right_axel_joint" type="revolute">
-        <parent link="base_link"/>
-        <child link="front_right_axel"/>
-        <origin xyz="-0.5543 ${-front_wheel_offset_y + 0.0319} 0" rpy="${pi/2} 0 0" />
-        <axis xyz="0 1 0"/>
-        <limit lower="${-pi/4}" upper="${pi/4}" velocity="100" effort="100"/>
-    </joint>
-    <link name="front_right_axel">
-        <visual>
-            <geometry>
-                <cylinder radius="0.005" length="0.0319"/>
-            </geometry>
-            <material name="red"/>
-        </visual>
-        <collision>
-            <geometry>
-                <sphere radius="0.005"/>
-            </geometry>
-        </collision>
-        <xacro:inertial_cylinder mass="0.005" length="0.0319" radius="0.005">
-            <origin xyz="0 0 0" rpy="0 0 0"/>
-        </xacro:inertial_cylinder>
-    </link>
-    <gazebo reference="front_right_axel">
-        <material>Gazebo/Red</material>
-    </gazebo>
-    <!-- FRONT RIGHT WHEEL LINK -->
-    <joint name="front_right_wheel_joint" type="fixed">
-        <parent link="front_right_axel"/>
-        <child link="front_right_wheel"/>
-        <origin xyz="0 0 0.0319" rpy="0 0 0" />
-        <axis xyz="0 0 -1"/>
-    </joint>
-    <link name="front_right_wheel">
-        <visual>
-            <geometry>
-                <cylinder radius="${front_wheel_radius}" length="${front_wheel_thickness}"/>
-            </geometry>
-            <material name="blue"/>
-        </visual>
-        <collision>
-            <geometry>
-                <sphere radius="${front_wheel_radius}"/>
-            </geometry>
-        </collision>
-        <xacro:inertial_cylinder mass="${wheel_mass}" length="${front_wheel_thickness}" radius="${front_wheel_radius}">
-            <origin xyz="0 0 0" rpy="0 0 0"/>
-        </xacro:inertial_cylinder>
-    </link>
-    <gazebo reference="front_right_wheel">
+    <gazebo reference="front_wheel">
         <material>Gazebo/Blue</material>
         <!-- <mu1 value="0.001"/>
@@ -181,8 +100,8 @@
     </gazebo>
     <!-- REAR LEFT WHEEL LINK -->
-    <joint name="rear_left_wheel_joint" type="continuous">
-        <parent link="base_link"/>
+    <joint name="rear_left_wheel_joint" type="fixed">
+        <parent link="rear_axel"/>
         <child link="rear_left_wheel"/>
-        <origin xyz="${rear_wheel_offset_x} ${rear_wheel_offset_y} 0" rpy="-${pi/2} 0 0" />
+        <origin xyz="0 0 ${rear_wheel_offset_y}" rpy="0 0 0" />
         <axis xyz="0 0 1"/>
     </joint>
@@ -206,9 +125,35 @@
         <material>Gazebo/Blue</material>
     </gazebo>
-<!-- REAR RIGHT WHEEL LINK -->
-    <joint name="rear_right_wheel_joint" type="continuous">
+    <!-- REAR AXEL LINK -->
+    <joint name="rear_axel_joint" type="continuous">
         <parent link="base_link"/>
+        <child link="rear_axel"/>
+        <origin xyz="${rear_wheel_offset_x} 0 0" rpy="${pi/2} 0 0" />
+        <axis xyz="0 0 -1"/>
+    </joint>
+    <link name="rear_axel">
+        <visual>
+            <geometry>
+                <cylinder radius="0.005" length="0.2202"/>
+            </geometry>
+            <material name="red"/>
+        </visual>
+        <collision>
+            <geometry>
+                <sphere radius="${rear_wheel_radius}"/>
+            </geometry>
+        </collision>
+        <xacro:inertial_cylinder mass="${wheel_mass}" length="0.2202" radius="0.005">
+            <origin xyz="0 0 0" rpy="0 0 0"/>
+        </xacro:inertial_cylinder>
+    </link>
+    <gazebo reference="rear_axel">
+        <material>Gazebo/Red</material>
+    </gazebo>
+    <!-- REAR RIGHT WHEEL LINK -->
+    <joint name="rear_right_wheel_joint" type="fixed">
+        <parent link="rear_axel"/>
         <child link="rear_right_wheel"/>
-        <origin xyz="${rear_wheel_offset_x} ${-rear_wheel_offset_y} 0" rpy="${pi/2} 0 0" />
+        <origin xyz="0 0 ${-rear_wheel_offset_y}" rpy="0 0 0" />
         <axis xyz="0 0 -1"/>
     </joint>
